Commit message: feat: refine instrument models and add placement controls

File: device-designer/models/opentrons_flex/opentrons_flex.urdf (robot description, URDF)
Before this commit: robot opentrons_flex_single_5_1000ul, 30 links, 29 joints
Links:
- removed link base
- removed link connections
- removed link deck
- removed link enclosure
- removed link frame
- removed link pipette
- removed link rear_power_switch
- removed link status_light
- removed link touchscreen
- removed link y_rails
- added link chassis; collision box size=0.05 0.06 0.71; collision box size=0.05 0.06 0.71
- added link deck_base; collision box size=0.847 0.614 0.014; visual mesh filename=meshes/deck_base.obj
- added link front_door_lower; collision box size=0.778 0.006 0.468; visual mesh filename=meshes/door_lower.obj
- added link front_door_upper; collision box size=0.778 0.006 0.204; visual mesh filename=meshes/door_upper.obj
- added link windows; collision box size=0.005 0.55 0.62; collision box size=0.005 0.55 0.62
- link asset_root: mass 88.5 -> None
- link carriage_x: geometry collision box size=0.18 0.12 0.4; visual mesh filename=meshes/cad_carriage.obj
- link carriage_z: geometry collision box size=0.061 0.09 0.28; visual mesh filename=meshes/pipette_8channel.obj
- link gantry_y: geometry collision box size=0.77 0.05 0.145; visual mesh filename=meshes/cad_gantry.obj
- link slot_a1: geometry collision box size=0.162 0.106 0.028; visual mesh filename=meshes/deck_insert.obj
- link slot_a2: geometry collision box size=0.162 0.106 0.028; visual mesh filename=meshes/deck_insert.obj
- link slot_a3: geometry collision box size=0.162 0.106 0.028; visual mesh filename=meshes/deck_insert.obj
- link slot_a4: geometry collision box size=0.146 0.102 0.017; visual mesh filename=meshes/staging_insert.obj
- link slot_b1: geometry collision box size=0.162 0.106 0.028; visual mesh filename=meshes/deck_insert.obj
- link slot_b2: geometry collision box size=0.162 0.106 0.028; visual mesh filename=meshes/deck_insert.obj
- link slot_b3: geometry collision box size=0.162 0.106 0.028; visual mesh filename=meshes/deck_insert.obj
- link slot_b4: geometry collision box size=0.146 0.102 0.017; visual mesh filename=meshes/staging_insert.obj
- link slot_c1: geometry collision box size=0.162 0.106 0.028; visual mesh filename=meshes/deck_insert.obj
- link slot_c2: geometry collision box size=0.162 0.106 0.028; visual mesh filename=meshes/deck_insert.obj
- link slot_c3: geometry collision box size=0.162 0.106 0.028; visual mesh filename=meshes/deck_insert.obj
- link slot_c4: geometry collision box size=0.146 0.102 0.017; visual mesh filename=meshes/staging_insert.obj
- link slot_d1: geometry collision box size=0.162 0.106 0.028; visual mesh filename=meshes/deck_insert.obj
- link slot_d2: geometry collision box size=0.162 0.106 0.028; visual mesh filename=meshes/deck_insert.obj
- link slot_d3: geometry collision box size=0.162 0.106 0.028; visual mesh filename=meshes/deck_insert.obj
- link slot_d4: geometry collision box size=0.146 0.102 0.017; visual mesh filename=meshes/staging_insert.obj
Joints:
- removed joint base_joint
- removed joint connections_joint
- removed joint deck_joint
- removed joint enclosure_joint
- removed joint frame_joint
- removed joint pipette_joint
- removed joint rear_power_rocker_joint
- removed joint status_light_joint
- removed joint touchscreen_joint
- removed joint y_rails_joint
- added joint chassis_joint: type fixed, parent asset_root, child chassis, origin xyz=0 0 0 rpy=0 0 0
- added joint deck_base_joint: type fixed, parent asset_root, child deck_base, origin xyz=0 0 0 rpy=0 0 0
- added joint front_door_fold_joint: type revolute, parent front_door_upper, child front_door_lower, origin xyz=0 0 -0.204 rpy=0 0 0, axis -1 0 0, limit lower=0 upper=3.14 effort=0 velocity=0
- added joint front_door_lift_joint: type revolute, parent asset_root, child front_door_upper, origin xyz=0 -0.333 0.761 rpy=0 0 0, axis -1 0 0, limit lower=0 upper=1.57 effort=0 velocity=0
- added joint windows_joint: type fixed, parent asset_root, child windows, origin xyz=0 0 0 rpy=0 0 0
- joint carriage_x_joint: limit lower=-0.24 upper=0.24 effort=0 velocity=0 -> lower=-0.28 upper=0.24 effort=0 velocity=0
- joint carriage_z_joint: axis 0 0 1 -> 0 0 -1; limit lower=0 upper=0.22 effort=0 velocity=0 -> lower=0 upper=0.2 effort=0 velocity=0; origin xyz=0 0 -0.22 rpy=0 0 0 -> xyz=-0.038 -0.113 0.09 rpy=0 0 0
- joint gantry_y_joint: limit lower=-0.21 upper=0.21 effort=0 velocity=0 -> lower=-0.1 upper=0.22 effort=0 velocity=0; origin xyz=0 0 0.64 rpy=0 0 0 -> xyz=0 0 0.51 rpy=0 0 0
- joint slot_a1_joint: origin xyz=-0.23 0.21 0.165 rpy=0 0 0 -> xyz=-0.177 0.11500000000000002 0.169 rpy=0 0 0
- joint slot_a2_joint: origin xyz=-0.05 0.21 0.165 rpy=0 0 0 -> xyz=-0.012999999999999984 0.11500000000000002 0.169 rpy=0 0 0
- joint slot_a3_joint: origin xyz=0.13 0.21 0.165 rpy=0 0 0 -> xyz=0.15100000000000002 0.11500000000000002 0.169 rpy=0 0 0
- joint slot_a4_joint: origin xyz=0.335 0.21 0.165 rpy=0 0 0 -> xyz=0.332 0.11500000000000002 0.169 rpy=0 0 0
- joint slot_b1_joint: origin xyz=-0.23 0.07 0.165 rpy=0 0 0 -> xyz=-0.177 0.008000000000000007 0.169 rpy=0 0 0
- joint slot_b2_joint: origin xyz=-0.05 0.07 0.165 rpy=0 0 0 -> xyz=-0.012999999999999984 0.008000000000000007 0.169 rpy=0 0 0
- joint slot_b3_joint: origin xyz=0.13 0.07 0.165 rpy=0 0 0 -> xyz=0.15100000000000002 0.008000000000000007 0.169 rpy=0 0 0
- joint slot_b4_joint: origin xyz=0.335 0.07 0.165 rpy=0 0 0 -> xyz=0.332 0.008000000000000007 0.169 rpy=0 0 0
- joint slot_c1_joint: origin xyz=-0.23 -0.07 0.165 rpy=0 0 0 -> xyz=-0.177 -0.09899999999999999 0.169 rpy=0 0 0
- joint slot_c2_joint: origin xyz=-0.05 -0.07 0.165 rpy=0 0 0 -> xyz=-0.012999999999999984 -0.09899999999999999 0.169 rpy=0 0 0
- joint slot_c3_joint: origin xyz=0.13 -0.07 0.165 rpy=0 0 0 -> xyz=0.15100000000000002 -0.09899999999999999 0.169 rpy=0 0 0
- joint slot_c4_joint: origin xyz=0.335 -0.07 0.165 rpy=0 0 0 -> xyz=0.332 -0.09899999999999999 0.169 rpy=0 0 0
- joint slot_d1_joint: origin xyz=-0.23 -0.21 0.165 rpy=0 0 0 -> xyz=-0.177 -0.206 0.169 rpy=0 0 0
- joint slot_d2_joint: origin xyz=-0.05 -0.21 0.165 rpy=0 0 0 -> xyz=-0.012999999999999984 -0.206 0.169 rpy=0 0 0
- joint slot_d3_joint: origin xyz=0.13 -0.21 0.165 rpy=0 0 0 -> xyz=0.15100000000000002 -0.206 0.169 rpy=0 0 0
- joint slot_d4_joint: origin xyz=0.335 -0.21 0.165 rpy=0 0 0 -> xyz=0.332 -0.206 0.169 rpy=0 0 0

Commit message: feat: refine Flex deck and toolhead from reference photos

File: device-designer/models/opentrons_flex/opentrons_flex.urdf (robot description, URDF)
Before this commit: robot opentrons_flex_8channel_photo_reference, 25 links, 24 joints
Links:
- removed link slot_a4
- removed link slot_b4
- removed link slot_c4
- removed link slot_d4
- added link gripper; collision box size=0.057 0.108 0.338; visual mesh filename=meshes/gripper_body.obj
- added link gripper_front; collision box size=0.037 0.028 0.133; visual mesh filename=meshes/gripper_front.obj
- added link gripper_rear; collision box size=0.037 0.028 0.133; visual mesh filename=meshes/gripper_rear.obj
- added link waste_bin; collision box size=0.215 0.087 0.043; visual mesh filename=meshes/waste_bin.obj
- link carriage_z: geometry collision box size=0.065 0.095 0.365; visual mesh filename=meshes/pipette_8channel.obj
- link slot_a1: geometry collision box size=0.244 0.106 0.028; visual mesh filename=meshes/deck_left.obj
- link slot_a3: geometry collision box size=0.27 0.106 0.028; visual mesh filename=meshes/deck_right.obj
- link slot_b1: geometry collision box size=0.244 0.106 0.028; visual mesh filename=meshes/deck_left.obj
- link slot_b3: geometry collision box size=0.27 0.106 0.028; visual mesh filename=meshes/deck_right.obj
- link slot_c1: geometry collision box size=0.244 0.106 0.028; visual mesh filename=meshes/deck_left.obj
- link slot_c3: geometry collision box size=0.27 0.106 0.028; visual mesh filename=meshes/deck_right.obj
- link slot_d1: geometry collision box size=0.244 0.106 0.028; visual mesh filename=meshes/deck_left.obj
- link slot_d3: geometry collision box size=0.27 0.106 0.028; visual mesh filename=meshes/deck_right.obj
Joints:
- removed joint slot_a4_joint
- removed joint slot_b4_joint
- removed joint slot_c4_joint
- removed joint slot_d4_joint
- added joint gripper_front_joint: type fixed, parent gripper, child gripper_front, origin xyz=0 0 0 rpy=0 0 0
- added joint gripper_rear_joint: type fixed, parent gripper, child gripper_rear, origin xyz=0 0 0 rpy=0 0 0
- added joint gripper_z_joint: type prismatic, parent carriage_x, child gripper, origin xyz=0.105 -0.105 0.09 rpy=0 0 0, axis 0 0 -1, limit lower=0 upper=0.14 effort=0 velocity=0
- added joint waste_bin_joint: type fixed, parent asset_root, child waste_bin, origin xyz=0.18 0.115 0.17 rpy=0 0 0
